File: 1090.sch (KiCad schematic (older format))
At the start: 94 parts, among them J1 Barrel_Jack, J2 J2, J3 J3, J4 J4, J5 J5, J6 J6, P1 PARALLEL_BUS_INTERFACE, U1 LM78M12, U2 LM78M05, U3 LM79M12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

Commit message: numerous changes to schematic and board files
Parts:
- J2, J3, J4, J5, J6: symbol 1090-rescue:EXPANSION_SLOT-expansion_slot-expansion_slot-1090-rescue -> 1090-rescue:EXPANSION_SLOT-expansion_slot-expansion_slot
- P1: symbol 1090-rescue:PARALLEL_BUS_INTERFACE-1090_parallel_bus_interface-1090-rescue -> 1090-rescue:PARALLEL_BUS_INTERFACE-1090_parallel_bus_interface
- S1: Manufacturer (none) -> C&K; Part # (none) -> E101J1AQE2; Vendor (none) -> Mouser
- U6: symbol 74xx_IEEE:74LS645 -> 1090-rescue:74LS645
Connections:
- net labels added: +10v, +15v_raw, -15v_raw
- wire segments 723 -> 730
- no-connect marks 0 -> 18
Other:
- moved on the sheet: TP3
Changed lines of the file:
@@
 $EndComp
 $Comp
-L 74xx_IEEE:74LS645 U6
+L 1090-rescue:74LS645 U6
 U 1 1 5CC95499
 P 7400 10100
@@
 Connection ~ 3200 9900
 $Comp
-L 1090-rescue:PARALLEL_BUS_INTERFACE-1090_parallel_bus_interface-1090-rescue P1
+L 1090-rescue:PARALLEL_BUS_INTERFACE-1090_parallel_bus_interface P1
 U 1 1 5CCE697D
 P 2450 8400
@@
 	16350 11150 16900 11150
 Wire Wire Line
-	16350 11250 16900 11250
+	16350 11250 16800 11250
 Wire Wire Line
 	16350 11350 16900 11350
@@
 F 1 "SW_SPST" H 2950 1850 50  0000 C CNN
 F 2 "1090:SPDT_Horiz_Rocker_Switch" H 2950 1750 50  0001 C CNN
-F 3 "~" H 2950 1750 50  0001 C CNN
+F 3 "https://www.ckswitches.com/media/1448/e_rocker.pdf" H 2950 1750 50  0001 C CNN
+F 4 "E101J1AQE2" H 2950 1750 50  0001 C CNN "Part #"
+F 5 "C&K" H 2950 1750 50  0001 C CNN "Manufacturer"
+F 6 "Mouser" H 2950 1750 50  0001 C CNN "Vendor"
 	1    2950 1750
 	1    0    0    -1
@@
 	7750 3350 8400 3350
 Connection ~ 7750 3350
-Wire Wire Line
-	7750 2300 8400 2300
 Connection ~ 7750 2300
-Wire Wire Line
-	7750 1350 8400 1350
 Connection ~ 7750 1350
 $Comp
@@
 	9550 3350 9900 3350
 Wire Wire Line
-	9000 2300 9550 2300
+	9000 2300 9200 2300
 Wire Wire Line
 	9550 2350 9550 2300
@@
 	9200 1900 9200 1950
 Connection ~ 9200 1950
-Wire Wire Line
-	9200 1950 7250 1950
 $Comp
 L Connector:TestPoint TP3
 U 1 1 61109848
-P 10550 2250
-F 0 "TP3" H 10500 2450 50  0000 L CNN
-F 1 "TestPoint" H 10608 2279 50  0001 L CNN
-F 2 "Connector_Pin:Pin_D1.0mm_L10.0mm" H 10750 2250 50  0001 C CNN
-F 3 "~" H 10750 2250 50  0001 C CNN
-	1    10550 2250
+P 9200 2300
+F 0 "TP3" H 9150 2500 50  0000 L CNN
+F 1 "TestPoint" H 9258 2329 50  0001 L CNN
+F 2 "Connector_Pin:Pin_D1.0mm_L10.0mm" H 9400 2300 50  0001 C CNN
+F 3 "~" H 9400 2300 50  0001 C CNN
+	1    9200 2300
 	1    0    0    -1
 $EndComp
@@
 Connection ~ 10350 2300
 Wire Wire Line
-	10350 2300 10550 2300
-Wire Wire Line
 	10700 2350 10700 2300
 Connection ~ 10700 2300
@@
 	4750 4450 7850 4450
 Connection ~ 4750 3850
-Wire Wire Line
-	10550 2250 10550 2300
-Connection ~ 10550 2300
-Wire Wire Line
-	10550 2300 10700 2300
 $Comp
 L Device:LED_ALT CR16
@@
 	1700 11000 1350 11000
 $Comp
-L 1090-rescue:EXPANSION_SLOT-expansion_slot-expansion_slot-1090-rescue J6
+L 1090-rescue:EXPANSION_SLOT-expansion_slot-expansion_slot J6
 U 1 1 5E4D3F8F
 P 21300 6550
@@
 $EndComp
 $Comp
-L 1090-rescue:EXPANSION_SLOT-expansion_slot-expansion_slot-1090-rescue J5
+L 1090-rescue:EXPANSION_SLOT-expansion_slot-expansion_slot J5
 U 1 1 5E4D4486
 P 18550 6550
@@
 $EndComp
 $Comp
-L 1090-rescue:EXPANSION_SLOT-expansion_slot-expansion_slot-1090-rescue J4
+L 1090-rescue:EXPANSION_SLOT-expansion_slot-expansion_slot J4
 U 1 1 5E4D4A57
 P 16150 6550
@@
 $EndComp
 $Comp
-L 1090-rescue:EXPANSION_SLOT-expansion_slot-expansion_slot-1090-rescue J3
+L 1090-rescue:EXPANSION_SLOT-expansion_slot-expansion_slot J3
 U 1 1 5E4D4D28
 P 13650 6550
@@
 $EndComp
 $Comp
-L 1090-rescue:EXPANSION_SLOT-expansion_slot-expansion_slot-1090-rescue J2
+L 1090-rescue:EXPANSION_SLOT-expansion_slot-expansion_slot J2
 U 1 1 5E4D50CD
 P 11200 6550
@@
 Wire Wire Line
 	4900 3350 4900 3450
+NoConn ~ 6750 12450
+NoConn ~ 6750 12850
+NoConn ~ 6750 12950
+NoConn ~ 5750 12950
+NoConn ~ 5750 12850
+NoConn ~ 5750 12450
+NoConn ~ 17900 13450
+NoConn ~ 17900 13350
+NoConn ~ 17900 12950
+NoConn ~ 19500 12950
+NoConn ~ 19500 13350
+NoConn ~ 19500 13450
+NoConn ~ 3050 9500
+NoConn ~ 3050 9600
+NoConn ~ 1700 11100
+NoConn ~ 1700 10800
+NoConn ~ 3650 3750
+NoConn ~ 2550 1850
+Connection ~ 9200 2300
+Wire Wire Line
+	9200 2300 9550 2300
+Wire Wire Line
+	10350 2300 10700 2300
+$Comp
+L power:VCC #PWR0141
+U 1 1 628EF6CF
+P 17200 11650
+F 0 "#PWR0141" H 17200 11500 50  0001 C CNN
+F 1 "VCC" H 17217 11823 50  0000 C CNN
+F 2 "" H 17200 11650 50  0001 C CNN
+F 3 "" H 17200 11650 50  0001 C CNN
+	1    17200 11650
+	1    0    0    -1
+$EndComp
+Wire Wire Line
+	17200 11650 17200 11700
+Wire Wire Line
+	17200 11700 16800 11700
+Wire Wire Line
+	16800 11700 16800 11250
+Connection ~ 16800 11250
+Wire Wire Line
+	16800 11250 16900 11250
+Wire Wire Line
+	7750 1350 8400 1350
+Wire Wire Line
+	7250 1950 8100 1950
+Wire Wire Line
+	7750 2300 8400 2300
+$Comp
+L Power_raw:+10v #+10v0101
+U 1 1 62C84876
+P 8100 1900
+F 0 "#+10v0101" H 8178 1962 50  0000 L CNN
+F 1 "+10v" H 8100 2000 50  0001 C CNN
+F 2 "" H 8100 1900 50  0001 C CNN
+F 3 "" H 8100 1900 50  0001 C CNN
+	1    8100 1900
+	1    0    0    -1
+$EndComp
+$Comp
+L Power_raw:+15v_raw #+15v0101
+U 1 1 62C862B5
+P 7750 1400
+F 0 "#+15v0101" H 7650 1550 50  0001 C CNN
+F 1 "+15v_raw" H 7828 1562 50  0000 L CNN
+F 2 "" H 7750 1400 50  0001 C CNN
+F 3 "" H 7750 1400 50  0001 C CNN
+	1    7750 1400
+	1    0    0    -1
+$EndComp
+$Comp
+L Power_raw:-15v_raw #-15v0101
+U 1 1 62C87CDE
+P 7750 3250
+F 0 "#-15v0101" H 7750 3250 50  0001 C CNN
+F 1 "-15v_raw" H 7828 3317 50  0000 L CNN
+F 2 "" H 7750 3250 50  0001 C CNN
+F 3 "" H 7750 3250 50  0001 C CNN
+	1    7750 3250
+	1    0    0    -1
+$EndComp
+Wire Wire Line
+	7750 1300 7750 1350
+Wire Wire Line
+	7750 3250 7750 3350
+Wire Wire Line
+	8100 1950 8100 1900
 Wire Bus Line
 	9300 5250 9300 12950
@@
 Wire Bus Line
 	22150 5250 22150 11250
+Connection ~ 8100 1950
+Wire Wire Line
+	8100 1950 9200 1950
 $EndSCHEMATC

Commit message: various board fixes
Changed lines of the file:
@@
 $EndComp
 Wire Wire Line
-	3200 9900 3200 10000
-Wire Wire Line
-	3050 10000 3200 10000
-Connection ~ 3200 10000
-Wire Wire Line
-	3200 10000 3200 10100
-Wire Wire Line
 	3050 10100 3200 10100
 Connection ~ 3200 10100
@@
 Wire Wire Line
 	3350 9350 3050 9350
-Text Notes 2200 9350 0    50   ~ 0
-/EXTENB
 Wire Wire Line
 	3500 12550 3500 9150
@@
 Text Label 1400 11000 0    50   ~ 0
 Pin47
-Text Label 10200 11200 0    50   ~ 0
+Text Label 10150 11200 0    50   ~ 0
 Pin47
-Text Label 10200 11350 0    50   ~ 0
+Text Label 10150 11350 0    50   ~ 0
 Pin39
-Text Label 12650 11350 0    50   ~ 0
+Text Label 12600 11350 0    50   ~ 0
 Pin39
-Text Label 15150 11350 0    50   ~ 0
+Text Label 15100 11350 0    50   ~ 0
 Pin39
-Text Label 17550 11350 0    50   ~ 0
+Text Label 17500 11350 0    50   ~ 0
 Pin39
-Text Label 20300 11350 0    50   ~ 0
+Text Label 20250 11350 0    50   ~ 0
 Pin39
-Text Label 12650 11200 0    50   ~ 0
+Text Label 12600 11200 0    50   ~ 0
 Pin47
-Text Label 15150 11200 0    50   ~ 0
+Text Label 15100 11200 0    50   ~ 0
 Pin47
-Text Label 17550 11200 0    50   ~ 0
+Text Label 17500 11200 0    50   ~ 0
 Pin47
-Text Label 20300 11200 0    50   ~ 0
+Text Label 20250 11200 0    50   ~ 0
 Pin47
 Text Label 2650 1750 0    50   ~ 0
@@
 Wire Wire Line
 	8100 1950 8100 1900
+Connection ~ 8100 1950
+Wire Wire Line
+	8100 1950 9200 1950
 Wire Bus Line
-	9300 5250 9300 12950
-Wire Bus Line
-	12050 5250 12050 11250
+	22150 5250 22150 11250
 Wire Bus Line
-	14500 5250 14500 11250
+	19400 5250 19400 11250
 Wire Bus Line
 	17000 5250 17000 11250
 Wire Bus Line
-	19400 5250 19400 11250
+	14500 5250 14500 11250
 Wire Bus Line
-	22150 5250 22150 11250
-Connection ~ 8100 1950
+	12050 5250 12050 11250
+Wire Bus Line
+	9300 5250 9300 12950
 Wire Wire Line
-	8100 1950 9200 1950
+	3200 10000 3200 10100
+Wire Wire Line
+	3200 9900 3200 10000
+Connection ~ 3200 10000
+Wire Wire Line
+	3050 10000 3200 10000
+Text Notes 2200 9350 0    50   ~ 0
+/EXTENB
 $EndSCHEMATC

Commit message: included many changes by pancio, update schematic and pcb to fix all DRC errors
Parts:
- C1, C18, C19, C20, C21, C22, C23, C24, C25, C26, C27, C28: footprint Capacitor_THT:C_Axial_L5.1mm_D3.1mm_P12.50mm_Horizontal -> 1090:C_Axial_L5.1mm_D3.1mm_P12.50mm_Horizontal
- C16: footprint Capacitor_THT:C_Axial_L5.1mm_D3.1mm_P15.00mm_Horizontal -> 1090:C_Axial_L5.1mm_D3.1mm_P12.50mm_Horizontal
- C3, C4, C7: footprint Capacitor_THT:CP_Radial_D25.0mm_P10.00mm_SnapIn -> 1090:CP_Radial_D22.0mm_P10.00mm_SnapIn
- C5, C6: footprint Capacitor_THT:CP_Radial_D16.0mm_P7.50mm -> 1090:CP_Radial_D13.0mm_P7.50mm
- CR1, CR2, CR3, CR4: footprint Diode_THT:D_5KP_P10.16mm_Horizontal -> 1090:D_5KP_P10.16mm_Horizontal
- CR15, CR16: footprint LED_THT:LED_Rectangular_W5.0mm_H2.0mm -> 1090:LED_D5.0mm_FlatTop
- S1: footprint 1090:SPDT_Horiz_Rocker_Switch -> footprints:E101J1ABE2
Connections:
- net labels added: rsvd
- wire segments 730 -> 737
Changed lines of the file:
@@
 F 0 "S1" H 2950 1985 50  0000 C CNN
 F 1 "SW_SPST" H 2950 1850 50  0000 C CNN
-F 2 "1090:SPDT_Horiz_Rocker_Switch" H 2950 1750 50  0001 C CNN
+F 2 "footprints:E101J1ABE2" H 2950 1750 50  0001 C CNN
 F 3 "https://www.ckswitches.com/media/1448/e_rocker.pdf" H 2950 1750 50  0001 C CNN
 F 4 "E101J1AQE2" H 2950 1750 50  0001 C CNN "Part #"
@@
 F 0 "CR3" H 5100 1500 50  0000 C CNN
 F 1 "D" H 5000 1475 50  0001 C CNN
-F 2 "Diode_THT:D_5KP_P10.16mm_Horizontal" H 5000 1600 50  0001 C CNN
+F 2 "1090:D_5KP_P10.16mm_Horizontal" H 5000 1600 50  0001 C CNN
 F 3 "~" H 5000 1600 50  0001 C CNN
 	1    5000 1600
@@
 F 0 "CR1" H 4600 1500 50  0000 C CNN
 F 1 "D" H 4500 1475 50  0001 C CNN
-F 2 "Diode_THT:D_5KP_P10.16mm_Horizontal" H 4500 1600 50  0001 C CNN
+F 2 "1090:D_5KP_P10.16mm_Horizontal" H 4500 1600 50  0001 C CNN
 F 3 "~" H 4500 1600 50  0001 C CNN
 	1    4500 1600
@@
 F 0 "CR2" H 4600 1800 50  0000 C CNN
 F 1 "D" H 4500 1775 50  0001 C CNN
-F 2 "Diode_THT:D_5KP_P10.16mm_Horizontal" H 4500 1900 50  0001 C CNN
+F 2 "1090:D_5KP_P10.16mm_Horizontal" H 4500 1900 50  0001 C CNN
 F 3 "~" H 4500 1900 50  0001 C CNN
 	1    4500 1900
@@
 F 0 "CR4" H 5100 1800 50  0000 C CNN
 F 1 "D" H 5000 1775 50  0001 C CNN
-F 2 "Diode_THT:D_5KP_P10.16mm_Horizontal" H 5000 1900 50  0001 C CNN
+F 2 "1090:D_5KP_P10.16mm_Horizontal" H 5000 1900 50  0001 C CNN
 F 3 "~" H 5000 1900 50  0001 C CNN
 	1    5000 1900
@@
 F 0 "CR15" V 7242 2382 50  0000 R CNN
 F 1 "LED_ALT" V 7197 2382 50  0001 R CNN
-F 2 "LED_THT:LED_Rectangular_W5.0mm_H2.0mm" H 7250 2500 50  0001 C CNN
+F 2 "1090:LED_D5.0mm_FlatTop" H 7250 2500 50  0001 C CNN
 F 3 "~" H 7250 2500 50  0001 C CNN
 	1    7250 2500
@@
 F 0 "C26" H 3950 2800 50  0000 L CNN
 F 1 ".01uF" H 3950 2700 50  0000 L CNN
-F 2 "Capacitor_THT:C_Axial_L5.1mm_D3.1mm_P12.50mm_Horizontal" H 4238 2650 50  0001 C CNN
+F 2 "1090:C_Axial_L5.1mm_D3.1mm_P12.50mm_Horizontal" H 4238 2650 50  0001 C CNN
 F 3 "~" H 4200 2800 50  0001 C CNN
 	1    4200 2800
@@
 F 0 "C25" H 3550 2800 50  0000 L CNN
 F 1 ".01uF" H 3550 2700 50  0000 L CNN
-F 2 "Capacitor_THT:C_Axial_L5.1mm_D3.1mm_P12.50mm_Horizontal" H 3838 2650 50  0001 C CNN
+F 2 "1090:C_Axial_L5.1mm_D3.1mm_P12.50mm_Horizontal" H 3838 2650 50  0001 C CNN
 F 3 "~" H 3800 2800 50  0001 C CNN
 	1    3800 2800
@@
 F 0 "C6" H 5200 2450 50  0000 L CNN
 F 1 "1500" H 5150 2350 50  0000 L CNN
-F 2 "Capacitor_THT:CP_Radial_D16.0mm_P7.50mm" H 5450 2400 50  0001 C CNN
+F 2 "1090:CP_Radial_D13.0mm_P7.50mm" H 5450 2400 50  0001 C CNN
 F 3 "~" H 5450 2400 50  0001 C CNN
 	1    5450 2400
@@
 F 0 "C3" H 5550 2000 50  0000 L CNN
 F 1 "3300" H 5500 1900 50  0000 L CNN
-F 2 "Capacitor_THT:CP_Radial_D25.0mm_P10.00mm_SnapIn" H 5800 1950 50  0001 C CNN
+F 2 "1090:CP_Radial_D22.0mm_P10.00mm_SnapIn" H 5800 1950 50  0001 C CNN
 F 3 "~" H 5800 1950 50  0001 C CNN
 	1    5800 1950
@@
 F 0 "C4" H 6000 2000 50  0000 L CNN
 F 1 "3300" H 5950 1900 50  0000 L CNN
-F 2 "Capacitor_THT:CP_Radial_D25.0mm_P10.00mm_SnapIn" H 6250 1950 50  0001 C CNN
+F 2 "1090:CP_Radial_D22.0mm_P10.00mm_SnapIn" H 6250 1950 50  0001 C CNN
 F 3 "~" H 6250 1950 50  0001 C CNN
 	1    6250 1950
@@
 F 0 "C7" V 5800 3350 50  0000 C CNN
 F 1 "3300" V 5500 3350 50  0000 C CNN
-F 2 "Capacitor_THT:CP_Radial_D25.0mm_P10.00mm_SnapIn" H 5650 3350 50  0001 C CNN
+F 2 "1090:CP_Radial_D22.0mm_P10.00mm_SnapIn" H 5650 3350 50  0001 C CNN
 F 3 "~" H 5650 3350 50  0001 C CNN
 	1    5650 3350
@@
 F 0 "C5" V 5250 3850 50  0000 C CNN
 F 1 "1500" V 4950 3850 50  0000 C CNN
-F 2 "Capacitor_THT:CP_Radial_D16.0mm_P7.50mm" H 5100 3850 50  0001 C CNN
+F 2 "1090:CP_Radial_D13.0mm_P7.50mm" H 5100 3850 50  0001 C CNN
 F 3 "~" H 5100 3850 50  0001 C CNN
 	1    5100 3850
@@
 F 0 "C1" H 3000 1900 50  0000 L CNN
 F 1 ".001uF" H 2900 1800 50  0000 L CNN
-F 2 "Capacitor_THT:C_Axial_L5.1mm_D3.1mm_P12.50mm_Horizontal" H 3200 1900 50  0001 C CNN
+F 2 "1090:C_Axial_L5.1mm_D3.1mm_P12.50mm_Horizontal" H 3200 1900 50  0001 C CNN
 F 3 "~" H 3200 1900 50  0001 C CNN
 	1    3200 1900
@@
 F 0 "C27" H 3350 1900 50  0000 L CNN
 F 1 ".01uF" H 3350 1800 50  0000 L CNN
-F 2 "Capacitor_THT:C_Axial_L5.1mm_D3.1mm_P12.50mm_Horizontal" H 3600 1900 50  0001 C CNN
+F 2 "1090:C_Axial_L5.1mm_D3.1mm_P12.50mm_Horizontal" H 3600 1900 50  0001 C CNN
 F 3 "~" H 3600 1900 50  0001 C CNN
 	1    3600 1900
@@
 F 0 "C28" H 3750 1900 50  0000 L CNN
 F 1 ".01uF" H 3750 1800 50  0000 L CNN
-F 2 "Capacitor_THT:C_Axial_L5.1mm_D3.1mm_P12.50mm_Horizontal" H 4000 1900 50  0001 C CNN
+F 2 "1090:C_Axial_L5.1mm_D3.1mm_P12.50mm_Horizontal" H 4000 1900 50  0001 C CNN
 F 3 "~" H 4000 1900 50  0001 C CNN
 	1    4000 1900
@@
 F 0 "C16" H 7850 3600 50  0000 L CNN
 F 1 ".22uF 50v" H 7800 3450 50  0000 L CNN
-F 2 "Capacitor_THT:C_Axial_L5.1mm_D3.1mm_P15.00mm_Horizontal" H 7750 3550 50  0001 C CNN
+F 2 "1090:C_Axial_L5.1mm_D3.1mm_P12.50mm_Horizontal" H 7750 3550 50  0001 C CNN
 F 3 "~" H 7750 3550 50  0001 C CNN
 	1    7750 3550
@@
 F 0 "C18" H 10100 2450 50  0000 L CNN
 F 1 ".01uF" H 10050 2350 50  0000 L CNN
-F 2 "Capacitor_THT:C_Axial_L5.1mm_D3.1mm_P12.50mm_Horizontal" H 10000 2450 50  0001 C CNN
+F 2 "1090:C_Axial_L5.1mm_D3.1mm_P12.50mm_Horizontal" H 10000 2450 50  0001 C CNN
 F 3 "~" H 10000 2450 50  0001 C CNN
 	1    10000 2450
@@
 F 0 "C19" H 10450 2450 50  0000 L CNN
 F 1 ".01uF" H 10400 2350 50  0000 L CNN
-F 2 "Capacitor_THT:C_Axial_L5.1mm_D3.1mm_P12.50mm_Horizontal" H 10350 2450 50  0001 C CNN
+F 2 "1090:C_Axial_L5.1mm_D3.1mm_P12.50mm_Horizontal" H 10350 2450 50  0001 C CNN
 F 3 "~" H 10350 2450 50  0001 C CNN
 	1    10350 2450
@@
 F 0 "C20" H 10800 2450 50  0000 L CNN
 F 1 ".01uF" H 10750 2350 50  0000 L CNN
-F 2 "Capacitor_THT:C_Axial_L5.1mm_D3.1mm_P12.50mm_Horizontal" H 10700 2450 50  0001 C CNN
+F 2 "1090:C_Axial_L5.1mm_D3.1mm_P12.50mm_Horizontal" H 10700 2450 50  0001 C CNN
 F 3 "~" H 10700 2450 50  0001 C CNN
 	1    10700 2450
@@
 F 0 "C21" H 11150 2450 50  0000 L CNN
 F 1 ".01uF" H 11100 2350 50  0000 L CNN
-F 2 "Capacitor_THT:C_Axial_L5.1mm_D3.1mm_P12.50mm_Horizontal" H 11050 2450 50  0001 C CNN
+F 2 "1090:C_Axial_L5.1mm_D3.1mm_P12.50mm_Horizontal" H 11050 2450 50  0001 C CNN
 F 3 "~" H 11050 2450 50  0001 C CNN
 	1    11050 2450
@@
 F 0 "C22" H 11500 2450 50  0000 L CNN
 F 1 ".01uF" H 11450 2350 50  0000 L CNN
-F 2 "Capacitor_THT:C_Axial_L5.1mm_D3.1mm_P12.50mm_Horizontal" H 11400 2450 50  0001 C CNN
+F 2 "1090:C_Axial_L5.1mm_D3.1mm_P12.50mm_Horizontal" H 11400 2450 50  0001 C CNN
 F 3 "~" H 11400 2450 50  0001 C CNN
 	1    11400 2450
@@
 F 0 "C23" H 11850 2450 50  0000 L CNN
 F 1 ".01uF" H 11800 2350 50  0000 L CNN
-F 2 "Capacitor_THT:C_Axial_L5.1mm_D3.1mm_P12.50mm_Horizontal" H 11750 2450 50  0001 C CNN
+F 2 "1090:C_Axial_L5.1mm_D3.1mm_P12.50mm_Horizontal" H 11750 2450 50  0001 C CNN
 F 3 "~" H 11750 2450 50  0001 C CNN
 	1    11750 2450
@@
 F 0 "C24" H 12200 2450 50  0000 L CNN
 F 1 ".01uF" H 12150 2350 50  0000 L CNN
-F 2 "Capacitor_THT:C_Axial_L5.1mm_D3.1mm_P12.50mm_Horizontal" H 12100 2450 50  0001 C CNN
+F 2 "1090:C_Axial_L5.1mm_D3.1mm_P12.50mm_Horizontal" H 12100 2450 50  0001 C CNN
 F 3 "~" H 12100 2450 50  0001 C CNN
 	1    12100 2450
@@
 F 0 "CR16" V 6742 1832 50  0000 R CNN
 F 1 "LED_ALT" V 6697 1832 50  0001 R CNN
-F 2 "LED_THT:LED_Rectangular_W5.0mm_H2.0mm" H 6750 1950 50  0001 C CNN
+F 2 "1090:LED_D5.0mm_FlatTop" H 6750 1950 50  0001 C CNN
 F 3 "~" H 6750 1950 50  0001 C CNN
 	1    6750 1950
@@
 Wire Wire Line
 	8100 1950 9200 1950
+Wire Wire Line
+	3200 10000 3200 10100
+Wire Wire Line
+	3200 9900 3200 10000
+Connection ~ 3200 10000
+Wire Wire Line
+	3050 10000 3200 10000
+Text Notes 2200 9350 0    50   ~ 0
+/EXTENB
+$Comp
+L power:+5V #PWR0142
+U 1 1 6162B249
+P 12500 1400
+F 0 "#PWR0142" H 12500 1250 50  0001 C CNN
+F 1 "+5V" H 12515 1573 50  0000 C CNN
+F 2 "" H 12500 1400 50  0001 C CNN
+F 3 "" H 12500 1400 50  0001 C CNN
+	1    12500 1400
+	1    0    0    -1
+$EndComp
+Wire Wire Line
+	12500 1400 12500 1500
+Wire Wire Line
+	12500 1500 12900 1500
+Text Label 12900 1500 0    50   ~ 0
++5V_REF
+Wire Wire Line
+	10400 11000 10150 11000
+Text Label 10150 11000 0    50   ~ 0
+rsvd
+Wire Wire Line
+	12850 11000 12600 11000
+Text Label 12600 11000 0    50   ~ 0
+rsvd
+Wire Wire Line
+	15350 11000 15100 11000
+Text Label 15100 11000 0    50   ~ 0
+rsvd
+Wire Wire Line
+	17750 11000 17500 11000
+Text Label 17500 11000 0    50   ~ 0
+rsvd
+Wire Wire Line
+	20500 11000 20250 11000
+Text Label 20250 11000 0    50   ~ 0
+rsvd
 Wire Bus Line
 	22150 5250 22150 11250
@@
 Wire Bus Line
 	9300 5250 9300 12950
-Wire Wire Line
-	3200 10000 3200 10100
-Wire Wire Line
-	3200 9900 3200 10000
-Connection ~ 3200 10000
-Wire Wire Line
-	3050 10000 3200 10000
-Text Notes 2200 9350 0    50   ~ 0
-/EXTENB
 $EndSCHEMATC
